File: Hardware/v01/ESP32_GPS_Motion_Shield.brd (EAGLE design)
At the start: 25.4 x 50.8 mm, 38 parts, among them J2 MICRO-SD_CARD_SOCKET, J6 3-PIN SMD, U1 LSM9DS1

Commit message: Reviewing for reds
Parts:
- added Q1, Q2: 4.3A/20V/54mΩ, SparkFun-DiscreteSemi:SOT23-3
- added R6: 10k, SparkFun-Resistors:0603
- moved R5 16.0 mm to (6.27, 14.6)
- moved LOGO1 6.73 mm to (7.43, 30.9)
- moved C5 3.17 mm to (11.8, 23.8), turned to 180 degrees
- moved C8 2.99 mm to (9.21, 23.3), turned to 270 degrees
- moved C4 1.29 mm to (9.21, 20.5)
- moved C6 0.43 mm to (11.1, 22.4), turned to 180 degrees
- moved LOGO2 0.37 mm to (7.70, 21.4)
Connections:
- removed net N$3: B1.17, J1.17
- removed net N$4: B1.16, J1.16
- removed net N$5: B1.19, J1.19
- removed net N$6: B1.10, J1.10
- removed net N$7: B1.14, J1.14
- new net 3.3V_B: B1.5, J1.5
- new net N$16: B1.7, J1.7
- new net N$43: B1.34, J3.14
- new net N$44: B1.35, J3.15
- new net VDD: C5.1, Q1.3, U1.22, U1.23
- new net VDDIO: C4.1, Q2.3, U1.1, U1.3
- new net VDDIO_CTRL: B1.14, J1.14, Q2.1, R5.1
- new net VDD_CTRL: B1.10, J1.10, Q1.1, R6.1
- net 3.3V: now also Q1.2, Q2.2, R6.2; no longer B1.5, C4.1, C5.1, J1.5, U1.1, U1.22, U1.23, U1.3
- net GND: now also J2.CD1
- net GPS_LED: now also B1.19, J1.19; no longer B1.7, J1.7
- net GPS_RX: now also B1.17, J1.17; no longer B1.34, J3.14
- net GPS_TX: now also B1.16, J1.16; no longer B1.35, J3.15
- net SD_CD: no longer R5.1
- net SD_DI: now also B1.26, J3.6; no longer B1.27, J3.7
- net SD_DO: now also B1.27, J3.7; no longer B1.26, J3.6
Routing:
- net GPS_LED: track 13.2 -> 45.3 mm
- net GPS_RX: track 23.7 -> 48.1 mm
- net VDDIO_CTRL: track 0.00 -> 24.0 mm, vias 0 -> 2
- net 3.3V: track 103.9 -> 82.4 mm, vias 5 -> 0
- net GPS_TX: track 28.3 -> 49.1 mm, vias 0 -> 1
- net VDD_CTRL: track 0.00 -> 17.9 mm, vias 0 -> 2
- net VDD: track 0.00 -> 7.54 mm
- net VDDIO: track 0.00 -> 5.69 mm
- net SD_CD: track 25.6 -> 21.6 mm
- net N$7: track 2.54 -> 0.00 mm
- net N$6: track 2.54 -> 0.00 mm
- net N$5: track 2.54 -> 0.00 mm
- net N$4: track 2.54 -> 0.00 mm
- net N$3: track 2.54 -> 0.00 mm
- net N$16: track 0.00 -> 2.54 mm
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Other:
- board text added: "v01"
- board text removed: "Motion Shield"
- board text removed: "v10"
