File: Hardware/v01/ESP32_GPS_Motion_Shield.sch (EAGLE design)
At the start: 38 parts, among them J2 MICRO-SD_CARD_SOCKET, J6 3-PIN SMD, U1 LSM9DS1

Commit message: Reviewing for reds
Parts:
- added Q1, Q2: 4.3A/20V/54mΩ, SparkFun-DiscreteSemi:MOSFET_PCH-IRLML2244
- added R6: 10k, SparkFun-Resistors:10KOHM-0603-1/10W-1%
Connections:
- removed net N$3: B1.39, J1.17
- removed net N$4: B1.32, J1.16
- removed net N$5: B1.37, J1.19
- removed net N$6: B1.27, J1.10
- removed net N$7: B1.34, J1.14
- new net 3.3V_B: B1.3V3@5, J1.5
- new net N$16: B1.13, J1.7
- new net N$43: B1.17, J3.14
- new net N$44: B1.16, J3.15
- new net VDD: C5.1, Q1.D, U1.VDD
- new net VDDIO: C4.1, Q2.D, U1.VDDIO
- new net VDDIO_CTRL: B1.34, J1.14, Q2.G, R5.1
- new net VDD_CTRL: B1.27, J1.10, Q1.G, R6.1
- net 3.3V: now also Q1.S, Q2.S, R6.2; no longer B1.3V3@5, C4.1, C5.1, J1.5, U1.VDD, U1.VDDIO
- net GND: now also J2.CD1
- net GPS_LED: now also B1.37, J1.19; no longer B1.13, J1.7
- net GPS_RX: now also B1.39, J1.17; no longer B1.17, J3.14
- net GPS_TX: now also B1.32, J1.16; no longer B1.16, J3.15
- net SD_CD: no longer R5.1
- net SD_DI: now also B1.19, J3.6; no longer B1.23, J3.7
- net SD_DO: now also B1.23, J3.7; no longer B1.19, J3.6
Other:
- note added: "v01"
- note removed: "v10"
- moved on the sheet: R5
